Commit message: changes to spawn point (WIP)

File: temp0.urdf (robot description, URDF)
Before this commit: robot pepe, 1 links, 0 joints
Links:
- added link 11, mass 2.8355394215966716; collision cylinder length=1.0840657599357362 radius=0.9124626462654255; visual cylinder length=1.0840657599357362 radius=0.9124626462654255
- added link 12, mass 2.8355394215966716; collision cylinder length=1.0840657599357362 radius=0.9124626462654255; visual cylinder length=1.0840657599357362 radius=0.9124626462654255
- added link 13, mass 2.8355394215966716; collision cylinder length=1.0840657599357362 radius=0.9124626462654255; visual cylinder length=1.0840657599357362 radius=0.9124626462654255
- link 0: mass 0.43729623076386187 -> 1.9985419975461454; geometry collision cylinder length=0.6364168237617274 radius=0.999794808390528; visual cylinder length=0.6364168237617274 radius=0.999794808390528
Joints:
- added joint 11_to_0: type revolute, parent 0, child 11, origin xyz=0.13180627528693292 0.9999 0.9267611180075409 rpy=3.274839276184391 1.0713722755009278 5.746925381524584, axis 1 0 0, limit lower=3.1415 upper=-3.1415 effort=1 velocity=1
- added joint 12_to_0: type revolute, parent 0, child 12, origin xyz=0.13180627528693292 0.9999 0.9267611180075409 rpy=4.9122589142765865 1.0713722755009278 5.746925381524584, axis 1 0 0, limit lower=3.1415 upper=-3.1415 effort=1 velocity=1
- added joint 13_to_0: type revolute, parent 0, child 13, origin xyz=0.13180627528693292 0.9999 0.9267611180075409 rpy=6.549678552368782 1.0713722755009278 5.746925381524584, axis 1 0 0, limit lower=3.1415 upper=-3.1415 effort=1 velocity=1

File: test.urdf (robot description, URDF)
Before this commit: robot pepe, 6 links, 5 joints
Links:
- removed link 33
- removed link 35
- added link 13, mass 1.370481291754875; collision cylinder length=0.4364168237617274 radius=0.999794808390528; visual cylinder length=0.4364168237617274 radius=0.999794808390528
- link 0: mass 0.004020374879162975 -> 2.3124089019564678; geometry collision cylinder length=0.8840657599357362 radius=0.9124626462654255; visual cylinder length=0.8840657599357362 radius=0.9124626462654255
- link 11: mass 0.6702422643953783 -> 1.370481291754875; geometry collision cylinder length=0.4364168237617274 radius=0.999794808390528; visual cylinder length=0.4364168237617274 radius=0.999794808390528
- link 22: mass 1.6076793590108298 -> 1.2674947805883765; geometry collision cylinder length=0.8268593568793257 radius=0.6985256060720479; visual cylinder length=0.8268593568793257 radius=0.6985256060720479
- link 24: mass 1.6076793590108298 -> 1.2674947805883765; geometry collision cylinder length=0.8268593568793257 radius=0.6985256060720479; visual cylinder length=0.8268593568793257 radius=0.6985256060720479
Joints:
- removed joint 24_to_11
- removed joint 33_to_22
- removed joint 35_to_24
- added joint 13_to_0: type revolute, parent 0, child 13, origin xyz=0.7760887543204691 0.4909697252385311 0.019209202782925816 rpy=18.18513722181167 1.7837898336827216 5.563482966679278, axis 1 0 0, limit lower=3.1415 upper=-3.1415 effort=1 velocity=1
- added joint 24_to_13: type revolute, parent 13, child 24, origin xyz=0.4224918593653373 0.362012300693504 0.1891445860003708 rpy=4.365391793148438 2.218919712129551 1.2202463958302825, axis 0 0 1, limit lower=3.1415 upper=-3.1415 effort=1 velocity=1
- joint 11_to_0: axis 0 0 1 -> 1 0 0; origin xyz=0.9999 0.5646409229007046 0.9493867399427927 rpy=4.068892381003681 5.465859679684793 4.687456269378126 -> xyz=0.7760887543204691 0.4909697252385311 0.019209202782925816 rpy=12.123424814541112 1.7837898336827216 5.563482966679278
- joint 22_to_11: origin xyz=0.9999 0.6646409229007045 0.9999 rpy=4.068892381003681 4.837541148966834 4.687456269378126 -> xyz=0.4224918593653373 0.362012300693504 0.1891445860003708 rpy=4.365391793148438 2.218919712129551 1.2202463958302825

Commit message: updated

File: temp0.urdf (robot description, URDF)
Before this commit: robot pepe, 31 links, 30 joints
Links:
- removed link 111
- removed link 121
- removed link 212
- removed link 215
- removed link 218
- removed link 22
- removed link 222
- removed link 225
- removed link 228
- removed link 25
- removed link 28
- removed link 310
- removed link 313
- removed link 314
- removed link 316
- removed link 317
- removed link 319
- removed link 320
- removed link 323
- removed link 324
- removed link 326
- removed link 327
- removed link 329
- removed link 33
- removed link 330
- removed link 34
- removed link 36
- removed link 37
- removed link 39
- added link 12, mass 0.006099295493998278; collision cylinder length=0.6950923040135429 radius=0.05284983803952781; visual cylinder length=0.6950923040135429 radius=0.05284983803952781
- added link 13, mass 0.006099295493998278; collision cylinder length=0.6950923040135429 radius=0.05284983803952781; visual cylinder length=0.6950923040135429 radius=0.05284983803952781
- added link 24, mass 0.2499729928016025; collision cylinder length=0.4149074603367672 radius=0.4379212166612972; visual cylinder length=0.4149074603367672 radius=0.4379212166612972
- link 0: mass 0.00020757668404297193 -> 0.007337481491887292; geometry collision cylinder length=0.566096535289482 radius=0.06423227800929465; visual cylinder length=0.566096535289482 radius=0.06423227800929465
- link 11: mass 0.14922753543433412 -> 0.006099295493998278; geometry collision cylinder length=0.6950923040135429 radius=0.05284983803952781; visual cylinder length=0.6950923040135429 radius=0.05284983803952781
Joints:
- removed joint 111_to_0
- removed joint 121_to_0
- removed joint 212_to_111
- removed joint 215_to_111
- removed joint 218_to_111
- removed joint 222_to_121
- removed joint 225_to_121
- removed joint 228_to_121
- removed joint 22_to_11
- removed joint 25_to_11
- removed joint 28_to_11
- removed joint 310_to_28
- removed joint 313_to_212
- removed joint 314_to_212
- removed joint 316_to_215
- removed joint 317_to_215
- removed joint 319_to_218
- removed joint 320_to_218
- removed joint 323_to_222
- removed joint 324_to_222
- removed joint 326_to_225
- removed joint 327_to_225
- removed joint 329_to_228
- removed joint 330_to_228
- removed joint 33_to_22
- removed joint 34_to_22
- removed joint 36_to_25
- removed joint 37_to_25
- removed joint 39_to_28
- added joint 12_to_0: type revolute, parent 0, child 12, origin xyz=0.41244013730074225 0.17398692755749967 0.8104611031487328 rpy=12.101967176663388 2.694689802316899 3.251427043631656, axis 0 1 0, limit lower=3.1415 upper=-3.1415 effort=1 velocity=1
- added joint 13_to_0: type revolute, parent 0, child 13, origin xyz=0.41244013730074225 0.17398692755749967 0.8104611031487328 rpy=16.135956235551184 2.694689802316899 3.251427043631656, axis 0 1 0, limit lower=3.1415 upper=-3.1415 effort=1 velocity=1
- added joint 24_to_0: type revolute, parent 0, child 24, origin xyz=0.7623505641157408 0.19244925293935772 0.9462391548407004 rpy=11.372530246323223 2.2227633803798414 4.830161811812665, axis 0 0 1, limit lower=3.1415 upper=-3.1415 effort=1 velocity=1
- joint 11_to_0: axis 0 0 1 -> 0 1 0; origin xyz=0.6256112701509253 0.9913149601512722 0.2636988888561938 rpy=12.534556007630535 2.749489669038799 6.188340482791822 -> xyz=0.41244013730074225 0.17398692755749967 0.8104611031487328 rpy=8.067978117775592 2.694689802316899 3.251427043631656

File: test.urdf (robot description, URDF)
Before this commit: robot pepe, 69 links, 68 joints
Links:
- removed link 118
- removed link 135
- removed link 152
- removed link 210
- removed link 214
- removed link 219
- removed link 22
- removed link 223
- removed link 227
- removed link 231
- removed link 236
- removed link 240
- removed link 244
- removed link 248
- removed link 253
- removed link 257
- removed link 26
- removed link 261
- removed link 265
- removed link 311
- removed link 312
- removed link 313
- removed link 315
- removed link 316
- removed link 317
- removed link 320
- removed link 321
- removed link 322
- removed link 324
- removed link 325
- removed link 326
- removed link 328
- removed link 329
- removed link 33
- removed link 330
- removed link 332
- removed link 333
- removed link 334
- removed link 337
- removed link 338
- removed link 339
- removed link 34
- removed link 341
- removed link 342
- removed link 343
- removed link 345
- removed link 346
- removed link 347
- removed link 349
- removed link 35
- removed link 350
- removed link 351
- removed link 354
- removed link 355
- removed link 356
- removed link 358
- removed link 359
- removed link 360
- removed link 362
- removed link 363
- removed link 364
- removed link 366
- removed link 367
- removed link 368
- removed link 37
- removed link 38
- removed link 39
- added link 12, mass 0.006099295493998278; collision cylinder length=0.6950923040135429 radius=0.05284983803952781; visual cylinder length=0.6950923040135429 radius=0.05284983803952781
- added link 13, mass 0.006099295493998278; collision cylinder length=0.6950923040135429 radius=0.05284983803952781; visual cylinder length=0.6950923040135429 radius=0.05284983803952781
- added link 24, mass 0.2499729928016025; collision cylinder length=0.4149074603367672 radius=0.4379212166612972; visual cylinder length=0.4149074603367672 radius=0.4379212166612972
- link 0: mass 0.00020757668404297193 -> 0.007337481491887292; geometry collision cylinder length=0.566096535289482 radius=0.06423227800929465; visual cylinder length=0.566096535289482 radius=0.06423227800929465
- link 11: mass 0.0886142984476594 -> 0.006099295493998278; geometry collision cylinder length=0.6950923040135429 radius=0.05284983803952781; visual cylinder length=0.6950923040135429 radius=0.05284983803952781
Joints:
- removed joint 118_to_0
- removed joint 135_to_0
- removed joint 152_to_0
- removed joint 210_to_11
- removed joint 214_to_11
- removed joint 219_to_118
- removed joint 223_to_118
- removed joint 227_to_118
- removed joint 22_to_11
- removed joint 231_to_118
- removed joint 236_to_135
- removed joint 240_to_135
- removed joint 244_to_135
- removed joint 248_to_135
- removed joint 253_to_152
- removed joint 257_to_152
- removed joint 261_to_152
- removed joint 265_to_152
- removed joint 26_to_11
- removed joint 311_to_210
- removed joint 312_to_210
- removed joint 313_to_210
- removed joint 315_to_214
- removed joint 316_to_214
- removed joint 317_to_214
- removed joint 320_to_219
- removed joint 321_to_219
- removed joint 322_to_219
- removed joint 324_to_223
- removed joint 325_to_223
- removed joint 326_to_223
- removed joint 328_to_227
- removed joint 329_to_227
- removed joint 330_to_227
- removed joint 332_to_231
- removed joint 333_to_231
- removed joint 334_to_231
- removed joint 337_to_236
- removed joint 338_to_236
- removed joint 339_to_236
- removed joint 33_to_22
- removed joint 341_to_240
- removed joint 342_to_240
- removed joint 343_to_240
- removed joint 345_to_244
- removed joint 346_to_244
- removed joint 347_to_244
- removed joint 349_to_248
- removed joint 34_to_22
- removed joint 350_to_248
- removed joint 351_to_248
- removed joint 354_to_253
- removed joint 355_to_253
- removed joint 356_to_253
- removed joint 358_to_257
- removed joint 359_to_257
- removed joint 35_to_22
- removed joint 360_to_257
- removed joint 362_to_261
- removed joint 363_to_261
- removed joint 364_to_261
- removed joint 366_to_265
- removed joint 367_to_265
- removed joint 368_to_265
- removed joint 37_to_26
- removed joint 38_to_26
- removed joint 39_to_26
- added joint 12_to_0: type revolute, parent 0, child 12, origin xyz=0.41244013730074225 0.17398692755749967 0.8104611031487328 rpy=12.101967176663388 2.694689802316899 3.251427043631656, axis 0 1 0, limit lower=3.1415 upper=-3.1415 effort=1 velocity=1
- added joint 13_to_0: type revolute, parent 0, child 13, origin xyz=0.41244013730074225 0.17398692755749967 0.8104611031487328 rpy=16.135956235551184 2.694689802316899 3.251427043631656, axis 0 1 0, limit lower=3.1415 upper=-3.1415 effort=1 velocity=1
- added joint 24_to_0: type revolute, parent 0, child 24, origin xyz=0.7623505641157408 0.19244925293935772 0.9462391548407004 rpy=11.372530246323223 2.2227633803798414 4.830161811812665, axis 0 0 1, limit lower=3.1415 upper=-3.1415 effort=1 velocity=1
- joint 11_to_0: axis 0 0 1 -> 0 1 0; origin xyz=0.5256112701509253 0.9913149601512722 0.2636988888561938 rpy=12.534556007630535 2.749489669038799 6.188340482791822 -> xyz=0.41244013730074225 0.17398692755749967 0.8104611031487328 rpy=8.067978117775592 2.694689802316899 3.251427043631656

Commit message: some modifications

File: temp0.urdf (robot description, URDF)
Before this commit: robot pepe, 5 links, 4 joints
Links:
- removed link 12
- removed link 13
- removed link 24
- added link 14, mass 0.04221066679325304; collision cylinder length=0.7440710708578562 radius=0.13437824354579808; visual cylinder length=0.7440710708578562 radius=0.13437824354579808
- added link 17, mass 0.04221066679325304; collision cylinder length=0.7440710708578562 radius=0.13437824354579808; visual cylinder length=0.7440710708578562 radius=0.13437824354579808
- added link 22, mass 0.6027566785865304; collision cylinder length=0.35049340519577266 radius=0.7398712534331663; visual cylinder length=0.35049340519577266 radius=0.7398712534331663
- added link 23, mass 0.6027566785865304; collision cylinder length=0.35049340519577266 radius=0.7398712534331663; visual cylinder length=0.35049340519577266 radius=0.7398712534331663
- added link 25, mass 0.6027566785865304; collision cylinder length=0.35049340519577266 radius=0.7398712534331663; visual cylinder length=0.35049340519577266 radius=0.7398712534331663
- added link 26, mass 0.6027566785865304; collision cylinder length=0.35049340519577266 radius=0.7398712534331663; visual cylinder length=0.35049340519577266 radius=0.7398712534331663
- added link 28, mass 0.6027566785865304; collision cylinder length=0.35049340519577266 radius=0.7398712534331663; visual cylinder length=0.35049340519577266 radius=0.7398712534331663
- added link 29, mass 0.6027566785865304; collision cylinder length=0.35049340519577266 radius=0.7398712534331663; visual cylinder length=0.35049340519577266 radius=0.7398712534331663
- link 0: mass 0.007337481491887292 -> 0.06824393164631085; geometry collision cylinder length=0.9936574974004084 radius=0.14785592289824545; visual cylinder length=0.9936574974004084 radius=0.14785592289824545
- link 11: mass 0.006099295493998278 -> 0.04221066679325304; geometry collision cylinder length=0.7440710708578562 radius=0.13437824354579808; visual cylinder length=0.7440710708578562 radius=0.13437824354579808
Joints:
- removed joint 12_to_0
- removed joint 13_to_0
- removed joint 24_to_0
- added joint 14_to_0: type revolute, parent 0, child 14, origin xyz=0.2968792383886708 0.6257359090449465 0.6350248467932161 rpy=10.395150176260316 4.544657722797063 3.5321751726918023, axis 1 0 0, limit lower=3.1415 upper=-3.1415 effort=1 velocity=1
- added joint 17_to_0: type revolute, parent 0, child 17, origin xyz=0.2968792383886708 0.6257359090449465 0.6350248467932161 rpy=13.860200235013755 4.544657722797063 3.5321751726918023, axis 1 0 0, limit lower=3.1415 upper=-3.1415 effort=1 velocity=1
- added joint 22_to_11: type revolute, parent 11, child 22, origin xyz=0.5699394173942979 0.5887691123488297 0.18950314772707033 rpy=7.7432642297688465 0.5725819966998213 3.894563894619473, axis 0 0 1, limit lower=3.1415 upper=-3.1415 effort=1 velocity=1
- added joint 23_to_11: type revolute, parent 11, child 23, origin xyz=0.5699394173942979 0.5887691123488297 0.18950314772707033 rpy=11.61489634465327 0.5725819966998213 3.894563894619473, axis 0 0 1, limit lower=3.1415 upper=-3.1415 effort=1 velocity=1
- added joint 25_to_14: type revolute, parent 14, child 25, origin xyz=0.5699394173942979 0.5887691123488297 0.18950314772707033 rpy=7.7432642297688465 0.5725819966998213 3.894563894619473, axis 0 0 1, limit lower=3.1415 upper=-3.1415 effort=1 velocity=1
- added joint 26_to_14: type revolute, parent 14, child 26, origin xyz=0.5699394173942979 0.5887691123488297 0.18950314772707033 rpy=11.61489634465327 0.5725819966998213 3.894563894619473, axis 0 0 1, limit lower=3.1415 upper=-3.1415 effort=1 velocity=1
- added joint 28_to_17: type revolute, parent 17, child 28, origin xyz=0.5699394173942979 0.5887691123488297 0.18950314772707033 rpy=7.7432642297688465 0.5725819966998213 3.894563894619473, axis 0 0 1, limit lower=3.1415 upper=-3.1415 effort=1 velocity=1
- added joint 29_to_17: type revolute, parent 17, child 29, origin xyz=0.5699394173942979 0.5887691123488297 0.18950314772707033 rpy=11.61489634465327 0.5725819966998213 3.894563894619473, axis 0 0 1, limit lower=3.1415 upper=-3.1415 effort=1 velocity=1
- joint 11_to_0: axis 0 1 0 -> 1 0 0; origin xyz=0.41244013730074225 0.17398692755749967 0.8104611031487328 rpy=8.067978117775592 2.694689802316899 3.251427043631656 -> xyz=0.2968792383886708 0.6257359090449465 0.6350248467932161 rpy=6.9301001175068775 4.544657722797063 3.5321751726918023

File: test.urdf (robot description, URDF)
Before this commit: robot pepe, 5 links, 4 joints
Links:
- added link 25, mass 0.010900650449650273; collision cylinder length=0.49716859859006846 radius=0.08354095296983455; visual cylinder length=0.49716859859006846 radius=0.08354095296983455
- link 0: mass 0.007337481491887292 -> 0.6807192926130667; geometry collision cylinder length=0.35049340519577266 radius=0.7862654057654562; visual cylinder length=0.35049340519577266 radius=0.7862654057654562
- link 11: mass 0.006099295493998278 -> 0.07013395251068648; geometry collision cylinder length=1.3319773915069566 radius=0.12946154763868378; visual cylinder length=1.3319773915069566 radius=0.12946154763868378
- link 12: mass 0.006099295493998278 -> 0.07013395251068648; geometry collision cylinder length=1.3319773915069566 radius=0.12946154763868378; visual cylinder length=1.3319773915069566 radius=0.12946154763868378
- link 13: mass 0.006099295493998278 -> 0.07013395251068648; geometry collision cylinder length=1.3319773915069566 radius=0.12946154763868378; visual cylinder length=1.3319773915069566 radius=0.12946154763868378
- link 24: mass 0.2499729928016025 -> 0.010900650449650273; geometry collision cylinder length=0.49716859859006846 radius=0.08354095296983455; visual cylinder length=0.49716859859006846 radius=0.08354095296983455
Joints:
- added joint 25_to_0: type revolute, parent 0, child 25, origin xyz=0.35710741877251195 0.5450486372767254 0.43291282129233777 rpy=24.667483750586925 4.230827455823204 1.1369956581674043, axis 0 1 0, limit lower=3.1415 upper=-3.1415 effort=1 velocity=1
- joint 11_to_0: origin xyz=0.41244013730074225 0.17398692755749967 0.8104611031487328 rpy=8.067978117775592 2.694689802316899 3.251427043631656 -> xyz=0.37960946265259965 0.06945360953443291 0.3995214680275563 rpy=2.5381404318221112 3.748373627327428 4.290494848505374
- joint 12_to_0: origin xyz=0.41244013730074225 0.17398692755749967 0.8104611031487328 rpy=12.101967176663388 2.694689802316899 3.251427043631656 -> xyz=0.37960946265259965 0.06945360953443291 0.3995214680275563 rpy=3.807210647733167 3.748373627327428 4.290494848505374
- joint 13_to_0: origin xyz=0.41244013730074225 0.17398692755749967 0.8104611031487328 rpy=16.135956235551184 2.694689802316899 3.251427043631656 -> xyz=0.37960946265259965 0.06945360953443291 0.3995214680275563 rpy=5.0762808636442225 3.748373627327428 4.290494848505374
- joint 24_to_0: axis 0 0 1 -> 0 1 0; origin xyz=0.7623505641157408 0.19244925293935772 0.9462391548407004 rpy=11.372530246323223 2.2227633803798414 4.830161811812665 -> xyz=0.35710741877251195 0.5450486372767254 0.43291282129233777 rpy=20.55623645882244 4.230827455823204 1.1369956581674043
