Commit message: Fix floating limbs: correct joint origin axis and use parent length
Root cause identified via diagnostic:
- Joint origin was offset in X-axis (xyz_1)
- URDF cylinders extend along Z-axis
- Child links were placed BESIDE parents, not at their endpoints
- Code used child's link_length instead of parent's

Fix:
- Added parent_link_length attribute to URDFLink class
- Store parent's link_length in child during expandLinks()
- Changed joint origin to use Z-axis offset with parent's length:
  xyz_3 = parent_len * 0.5 (instead of xyz_1 = child_len * 0.5)

Verified:
- Before: Child at (0.57, 0, 2.0) - floating beside parent
- After: Child at (0.05, 0, 2.325) - attached at parent's endpoint

File: diagnostic_creature.urdf (robot description, URDF)
Before this commit: robot pepe, 2 links, 1 joints
Joints:
- joint 11_to_0: origin xyz=0.5700000000000001 0.0 0.0 rpy=0.0 0.0 0.0 -> xyz=0.05 0.0 0.325 rpy=0.0 0.0 0.0
