Commit message: updated code

File: test.urdf (robot description, URDF)
Before this commit: robot pepe, 6 links, 5 joints
Links:
- removed link 12
- removed link 13
- removed link 24
- removed link 25
- added link 22, mass 0.5234417116730592; collision sphere radius=0.49995000000000006; visual sphere radius=0.49995000000000006
- added link 33, mass 0.01978641278714489; collision box size=0.3381235927324284 0.3421060802331988 0.1710530401165994; visual box size=0.3381235927324284 0.3421060802331988 0.1710530401165994
- added link 44, mass 0.4768211375414801; collision sphere radius=0.484643393249023; visual sphere radius=0.484643393249023
- added link 55, mass 0.0014497990606651297; collision cylinder length=0.1 radius=0.0679327147985184; visual cylinder length=0.1 radius=0.0679327147985184
- link 0: mass 0.6807192926130667 -> 0.002160390956282217; geometry collision cylinder length=0.27506951976267324 radius=0.05; visual cylinder length=0.27506951976267324 radius=0.05
- link 11: mass 0.07013395251068648 -> 0.0037933779329377233; geometry collision box size=0.534229208405772 0.11916925933410089 0.05958462966705044; visual box size=0.534229208405772 0.11916925933410089 0.05958462966705044
Joints:
- removed joint 12_to_0
- removed joint 13_to_0
- removed joint 24_to_0
- removed joint 25_to_0
- added joint 22_to_0: type revolute, parent 0, child 22, origin xyz=0.2 -0.2 0.1875347598813366 rpy=0.0 6.282556988648868 2.620525897571362, axis 1 0 0, limit lower=-3.1415 upper=3.1415 effort=10 velocity=5
- added joint 33_to_0: type revolute, parent 0, child 33, origin xyz=0.30369743571641494 -0.30000000000000004 0.24828475077223128 rpy=17.453475909377346 4.64226481617223 1.78861107924055, axis 1 0 0, limit lower=-3.1415 upper=3.1415 effort=10 velocity=5
- added joint 44_to_33: type revolute, parent 33, child 44, origin xyz=0.18293798684270418 0.03110990088968571 0.23685050336547714 rpy=1.129583493435578 1.9563291147378916 0.0, axis 0 0 1, limit lower=-3.1415 upper=3.1415 effort=10 velocity=5
- added joint 55_to_0: type revolute, parent 0, child 55, origin xyz=0.44479921514298226 -0.10003000000000001 0.2544435186940844 rpy=9.886982067921897 0.0 1.9901283336372813, axis 1 0 0, limit lower=-3.1415 upper=3.1415 effort=10 velocity=5
- joint 11_to_0: axis 0 1 0 -> 0 0 1; limit lower=3.1415 upper=-3.1415 effort=1 velocity=1 -> lower=-3.1415 upper=3.1415 effort=10 velocity=5; origin xyz=0.37960946265259965 0.06945360953443291 0.3995214680275563 rpy=2.5381404318221112 3.748373627327428 4.290494848505374 -> xyz=0.1 0.0979193793906658 0.22015953949526637 rpy=0.6128253082028159 0.0 3.9794648135417843
